File: board_design/CEC_PCB/CEC_PCB.kicad_pcb (KiCad board)
At the start: 4 copper layers, 50 x 40 mm, 19 parts, among them J1 HDMI_A, J2 HDMI_A, J3 Conn_02x12_Odd_Even, J4 Conn_02x12_Odd_Even, J5 Conn_01x06_Pin, Q1 BSS138, U1 XC6206PxxxMR

Commit message: Final PCB touches
Routing:
- net GND: track 19.3 -> 6.94 mm, vias 48 -> 46
- net /D0S: track 38.0 -> 39.1 mm
Changed lines of the file:
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@@
     (title "ATmega32u4 CEC capable device")
     (date "2024-03-19")
-    (rev "0.1")
+    (rev "1.0")
   )
   (layers
@@
   (segment (start 139 77.4) (end 139 80.1) (width 0.3) (layer "F.Cu") (net 1))
   (segment (start 158.5 81.8) (end 150.2 81.8) (width 0.3) (layer "F.Cu") (net 1))
-  (segment (start 163.2 78.74) (end 161.96 77.5) (width 0.3) (layer "F.Cu") (net 1))
   (segment (start 136 107.6) (end 138 109.6) (width 0.3) (layer "F.Cu") (net 1))
   (segment (start 148.4 109.2) (end 147.570049 108.370049) (width 0.3) (layer "F.Cu") (net 1))
   (segment (start 144.480049 105.58) (end 144.490049 105.59) (width 0.3) (layer "F.Cu") (net 1))
+  (segment (start 163.2 78.74) (end 161.96 77.5) (width 0.3) (layer "F.Cu") (net 1))
   (segment (start 138.2 80.9) (end 138.2 84.792894) (width 0.3) (layer "F.Cu") (net 1))
   (segment (start 136 86.992894) (end 136 107.6) (width 0.3) (layer "F.Cu") (net 1))
@@
   (segment (start 139 113.56) (end 139 110.6) (width 0.3) (layer "F.Cu") (net 1))
   (segment (start 138.65 105.75) (end 140.2 104.2) (width 0.3) (layer "F.Cu") (net 1))
+  (segment (start 163.2 79.95) (end 163.2 78.74) (width 0.3) (layer "F.Cu") (net 1))
   (segment (start 149.05 86.75) (end 148.5 86.2) (width 0.3) (layer "F.Cu") (net 1))
   (segment (start 138.65 107.6) (end 138.65 105.75) (width 0.3) (layer "F.Cu") (net 1))
@@
   (segment (start 139 110.6) (end 138 109.6) (width 0.3) (layer "F.Cu") (net 1))
   (segment (start 163.65 106) (end 163.65 106.190049) (width 0.3) (layer "F.Cu") (net 1))
-  (segment (start 163.2 79.7) (end 163.2 78.74) (width 0.3) (layer "F.Cu") (net 1))
   (via (at 138 109.6) (size 0.8) (drill 0.4) (layers "F.Cu" "B.Cu") (net 1))
   (via (at 150.2 81.8) (size 0.8) (drill 0.4) (layers "F.Cu" "B.Cu") (net 1))
@@
   (via (at 158.5 81.8) (size 0.8) (drill 0.4) (layers "F.Cu" "B.Cu") (net 1))
   (via (at 138.65 107.6) (size 0.8) (drill 0.4) (layers "F.Cu" "B.Cu") (net 1))
-  (via (at 163.2 79.7) (size 0.8) (drill 0.4) (layers "F.Cu" "B.Cu") (net 1))
+  (via (at 163.2 79.95) (size 0.8) (drill 0.4) (layers "F.Cu" "B.Cu") (net 1))
   (segment (start 138 109.6) (end 138 108.25) (width 0.3) (layer "B.Cu") (net 1))
   (segment (start 148.5 86.2) (end 149.2 85.5) (width 0.3) (layer "B.Cu") (net 1))
@@
   (segment (start 137.040049 113.56) (end 137.040049 112.2) (width 0.5) (layer "F.Cu") (net 4))
   (segment (start 135.890049 80) (end 137.040049 78.85) (width 0.5) (layer "F.Cu") (net 4))
-  (segment (start 164.5 77.5) (end 166.9 77.5) (width 0.3) (layer "F.Cu") (net 4))
-  (segment (start 168.5 105.38) (end 171.04 105.38) (width 0.5) (layer "F.Cu") (net 4))
   (segment (start 156.83 91.32) (end 156.8 91.35) (width 0.5) (layer "F.Cu") (net 4))
   (segment (start 137.040049 112.2) (end 135.840049 111) (width 0.5) (layer "F.Cu") (net 4))
-  (segment (start 155.81 110.46) (end 155.85 110.5) (width 0.5) (layer "F.Cu") (net 4))
-  (segment (start 151 110.46) (end 153.54 110.46) (width 0.5) (layer "F.Cu") (net 4))
   (segment (start 135.840049 111) (end 135.540049 111) (width 0.5) (layer "F.Cu") (net 4))
   (segment (start 135.55 80) (end 135.890049 80) (width 0.5) (layer "F.Cu") (net 4))
   (segment (start 159.840049 90.7975) (end 159.902549 90.86) (width 0.5) (layer "F.Cu") (net 4))
-  (segment (start 153.54 110.46) (end 155.81 110.46) (width 0.5) (layer "F.Cu") (net 4))
-  (segment (start 168.5 107.92) (end 171.04 107.92) (width 0.5) (layer "F.Cu") (net 4))
   (via (at 149.15 80.8) (size 0.8) (drill 0.4) (layers "F.Cu" "B.Cu") (free) (net 4))
   (via (at 159.2 89.6) (size 0.8) (drill 0.4) (layers "F.Cu" "B.Cu") (free) (net 4))
@@
   (via (at 140.4 92.35) (size 0.8) (drill 0.4) (layers "F.Cu" "B.Cu") (free) (net 4))
   (via (at 148 104.35) (size 0.8) (drill 0.4) (layers "F.Cu" "B.Cu") (free) (net 4))
-  (via (at 166.9 77.5) (size 0.8) (drill 0.4) (layers "F.Cu" "B.Cu") (free) (net 4))
   (via (at 140.4 101.9) (size 0.8) (drill 0.4) (layers "F.Cu" "B.Cu") (free) (net 4))
   (via (at 142.6 95.8) (size 0.8) (drill 0.4) (layers "F.Cu" "B.Cu") (free) (net 4))
@@
   (via (at 132 103) (size 0.8) (drill 0.4) (layers "F.Cu" "B.Cu") (free) (net 4))
   (via (at 144.7 104.35) (size 0.8) (drill 0.4) (layers "F.Cu" "B.Cu") (free) (net 4))
-  (via (at 155.85 110.5) (size 0.8) (drill 0.4) (layers "F.Cu" "B.Cu") (free) (net 4))
   (via (at 165 108.55) (size 0.8) (drill 0.4) (layers "F.Cu" "B.Cu") (free) (net 4))
   (via (at 157 95) (size 0.8) (drill 0.4) (layers "F.Cu" "B.Cu") (free) (net 4))
@@
   (segment (start 139.540049 113.56) (end 139.540049 111.459999) (width 0.2) (layer "B.Cu") (net 19))
   (segment (start 139.815049 111.184999) (end 139.815049 107.465792) (width 0.2) (layer "B.Cu") (net 19))
+  (segment (start 148.55 106.660661) (end 148.55 109.550049) (width 0.3) (layer "B.Cu") (net 20))
+  (segment (start 148.370049 81.58) (end 148.370049 84.779951) (width 0.3) (layer "B.Cu") (net 20))
+  (segment (start 148.370049 84.779951) (end 147.1 86.05) (width 0.3) (layer "B.Cu") (net 20))
+  (segment (start 147.1 105.210661) (end 148.55 106.660661) (width 0.3) (layer "B.Cu") (net 20))
+  (segment (start 144.540049 77.36) (end 144.540049 77.75) (width 0.3) (layer "B.Cu") (net 20))
   (segment (start 147.1 86.05) (end 147.1 105.210661) (width 0.3) (layer "B.Cu") (net 20))
   (segment (start 144.540049 77.75) (end 148.370049 81.58) (width 0.3) (layer "B.Cu") (net 20))
-  (segment (start 144.540049 77.36) (end 144.540049 77.75) (width 0.3) (layer "B.Cu") (net 20))
-  (segment (start 148.320049 109.78) (end 144.540049 113.56) (width 0.3) (layer "B.Cu") (net 20))
-  (segment (start 148.370049 81.58) (end 148.370049 84.779951) (width 0.3) (layer "B.Cu") (net 20))
-  (segment (start 148.370049 84.779951) (end 147.1 86.05) (width 0.3) (layer "B.Cu") (net 20))
-  (segment (start 148.320049 106.43071) (end 148.320049 109.78) (width 0.3) (layer "B.Cu") (net 20))
-  (segment (start 147.1 105.210661) (end 148.320049 106.43071) (width 0.3) (layer "B.Cu") (net 20))
+  (segment (start 148.55 109.550049) (end 144.540049 113.56) (width 0.3) (layer "B.Cu") (net 20))
   (segment (start 143.040049 77.36) (end 143.040049 81.440049) (width 0.3) (layer "F.Cu") (net 21))
   (segment (start 144.9 93.75) (end 144.9 96.85) (width 0.3) (layer "F.Cu") (net 21))
@@
   (segment (start 144.9 99.8) (end 144.9 102.65) (width 0.3) (layer "F.Cu") (net 21))
   (segment (start 145.35 99.35) (end 144.9 99.8) (width 0.3) (layer "F.Cu") (net 21))
-  (segment (start 139.4 88.984645) (end 139.4 105.11) (width 0.3) (layer "B.Cu") (net 22))
-  (segment (start 139.4 105.11) (end 141.540049 107.250049) (width 0.3) (layer "B.Cu") (net 22))
+  (segment (start 140.45 100.789339) (end 139.65 101.589339) (width 0.3) (layer "B.Cu") (net 22))
   (segment (start 141.540049 77.36) (end 141.540049 86.844596) (width 0.3) (layer "B.Cu") (net 22))
+  (segment (start 139.65 97.55) (end 140.45 98.35) (width 0.3) (layer "B.Cu") (net 22))
+  (segment (start 139.65 92.660661) (end 140.45 93.460661) (width 0.3) (layer "B.Cu") (net 22))
+  (segment (start 139.65 88.734645) (end 139.65 92.660661) (width 0.3) (layer "B.Cu") (net 22))
+  (segment (start 139.65 95.9) (end 139.65 97.55) (width 0.3) (layer "B.Cu") (net 22))
+  (segment (start 140.45 98.35) (end 140.45 100.789339) (width 0.3) (layer "B.Cu") (net 22))
+  (segment (start 139.65 105.36) (end 141.540049 107.250049) (width 0.3) (layer "B.Cu") (net 22))
+  (segment (start 140.45 95.1) (end 139.65 95.9) (width 0.3) (layer "B.Cu") (net 22))
   (segment (start 141.540049 107.250049) (end 141.540049 113.56) (width 0.3) (layer "B.Cu") (net 22))
-  (segment (start 141.540049 86.844596) (end 139.4 88.984645) (width 0.3) (layer "B.Cu") (net 22))
+  (segment (start 139.65 101.589339) (end 139.65 105.36) (width 0.3) (layer "B.Cu") (net 22))
+  (segment (start 141.540049 86.844596) (end 139.65 88.734645) (width 0.3) (layer "B.Cu") (net 22))
+  (segment (start 140.45 93.460661) (end 140.45 95.1) (width 0.3) (layer "B.Cu") (net 22))
   (segment (start 139.2 84.7) (end 139.2 80.790049) (width 0.3) (layer "F.Cu") (net 23))
   (segment (start 140 113.56) (end 140 110.239339) (width 0.3) (layer "F.Cu") (net 23))
